Commit message: feat(eval): ground LIBERO policies in calibrated RGB-D

File: dimos/benchmark/libero_pro/panda.urdf (robot description, URDF)
Before this commit: robot panda, 10 links, 9 joints
Links:
- added link tcp
Joints:
- added joint tcp_fixed: type fixed, parent right_hand, child tcp, origin xyz=0 0 0.097 rpy=0 0 -1.57079632679

Commit message: feat(manipulation): add grounded realtime pick and place

File: dimos/benchmark/libero_pro/panda.urdf (robot description, URDF)
Before this commit: robot panda, 11 links, 10 joints
Links:
- link link1: geometry collision cylinder length=0.283 radius=0.06
- link link2: geometry collision cylinder length=0.12 radius=0.06
- link link3: geometry collision cylinder length=0.15 radius=0.06
- link link4: geometry collision cylinder length=0.12 radius=0.06
- link link5: geometry collision cylinder length=0.10 radius=0.06
- link link6: geometry collision cylinder length=0.08 radius=0.05
- link link7: geometry collision cylinder length=0.14 radius=0.04
- link right_hand: geometry collision box size=0.10 0.10 0.12
