Commit message: alfred: update the D455 camera_joint to the re-angled mount
The camera was physically re-angled between 2026-08-16 and 2026-08-18, so the URDF's
pitch described hardware that no longer exists. Scored against a point-lio voxel map on
drive_2026-08-18_23-05-04.db, the old angle puts the floor at z=+1.80 while the new one
lands it at z=-0.40, matching the lidar exactly (IoU 0.019 -> 0.107).

File: dimos/robot/diy/alfred/alfred.urdf (robot description, URDF)
Before this commit: robot alfred, 19 links, 18 joints
Joints:
- joint camera_joint: origin xyz=-0.2518 -0.2736 0.48 rpy=-0.0097 -0.4020 -3.1030 -> xyz=-0.2518 -0.2736 0.42 rpy=-0.0097 0.1571 -3.1030

Commit message: alfred: correct the camera subtree to the D455 extrinsics
The child offsets were D435 values: a 50 mm stereo baseline where the D455 reports
95 mm, and colour on the wrong side of the left imager. The RealSense module
publishes the device extrinsics at runtime, so only the rerun model was wrong.
Values read back off the device in the 2026-08-25 spin recording.

File: dimos/robot/diy/alfred/alfred.urdf (robot description, URDF)
Before this commit: robot alfred, 19 links, 18 joints
Joints:
- joint camera_accel_joint: origin xyz=-0.0117 -0.0055 0.0051 rpy=0 0 0 -> xyz=-0.016 -0.0302 0.0074 rpy=0 0 0
- joint camera_color_joint: origin xyz=-0.0004 0.0149 -0.0002 rpy=0 0 0 -> xyz=-0.0004 -0.0592 0.0001 rpy=0 0 0
- joint camera_infra2_joint: origin xyz=0 -0.0499 0 rpy=0 0 0 -> xyz=0 -0.0949 0 rpy=0 0 0

Commit message: alfred: recalibrate the D455 mount off the 2026-08-25 spin
Roll, pitch and height come from the spin recording scored against the Mid-360;
yaw, x and y stay as measured, since a spin in place leaves those axes flat.
Median depth-to-lidar distance improves 8.4 cm to 8.1 cm, inliers 35% to 38%.
The blueprint constant carries the same pose as the urdf joint.

File: dimos/robot/diy/alfred/alfred.urdf (robot description, URDF)
Before this commit: robot alfred, 19 links, 18 joints
Joints:
- joint camera_joint: origin xyz=-0.2518 -0.2736 0.42 rpy=-0.0097 0.1571 -3.1030 -> xyz=-0.2518 -0.2736 0.4292 rpy=0.0512 0.1592 -3.1030

Commit message: alfred: rework urdf for the rebuilt sensor layout
D435i replaces the D455: upside-down on a 40mm rail at the rear center
(photo-estimated, pending spin calibration). Mast moved to the front
center. Mid-360 calibrated transform unchanged.

File: dimos/robot/diy/alfred/alfred.urdf (robot description, URDF)
Before this commit: robot alfred, 19 links, 18 joints
Links:
- link camera_link: geometry visual box size=0.025 0.090 0.025
- link mast_link: geometry collision box size=0.10 0.20 0.65; visual box size=0.10 0.20 0.65
Joints:
- joint camera_accel_joint: origin xyz=-0.016 -0.0302 0.0074 rpy=0 0 0 -> xyz=-0.0112 -0.0055 0.0051 rpy=0 0 0
- joint camera_color_joint: origin xyz=-0.0004 -0.0592 0.0001 rpy=0 0 0 -> xyz=0 -0.015 0 rpy=0 0 0
- joint camera_infra2_joint: origin xyz=0 -0.0949 0 rpy=0 0 0 -> xyz=0 -0.050 0 rpy=0 0 0
- joint camera_joint: origin xyz=-0.2518 -0.2736 0.4292 rpy=0.0512 0.1592 -3.1030 -> xyz=-0.13 0 0.391 rpy=3.1415927 0 3.1415927
- joint mast_joint: origin xyz=-0.04 0 0.331 rpy=0 0 0 -> xyz=0.21 0 0.331 rpy=0 0 0

Commit message: alfred: switch to the mast D455, measured off the base-height photo

File: dimos/robot/diy/alfred/alfred.urdf (robot description, URDF)
Before this commit: robot alfred, 19 links, 18 joints
Links:
- added link d455_accel_frame
- added link d455_accel_optical_frame
- added link d455_color_frame
- added link d455_color_optical_frame
- added link d455_depth_frame
- added link d455_depth_optical_frame
- added link d455_infra1_frame
- added link d455_infra1_optical_frame
- added link d455_infra2_frame
- added link d455_infra2_optical_frame
- added link d455_link; visual box size=0.026 0.124 0.029
- link mast_link: geometry collision box size=0.10 0.20 1.68; visual box size=0.10 0.20 1.68
Joints:
- added joint d455_accel_joint: type fixed, parent d455_link, child d455_accel_frame, origin xyz=-0.0160 -0.0302 0.0074 rpy=0 0 0
- added joint d455_accel_optical_joint: type fixed, parent d455_accel_frame, child d455_accel_optical_frame, origin xyz=0 0 0 rpy=-1.5707963 0 -1.5707963
- added joint d455_color_joint: type fixed, parent d455_link, child d455_color_frame, origin xyz=0 -0.029 0 rpy=0 0 0
- added joint d455_color_optical_joint: type fixed, parent d455_color_frame, child d455_color_optical_frame, origin xyz=0 0 0 rpy=-1.5707963 0 -1.5707963
- added joint d455_depth_joint: type fixed, parent d455_link, child d455_depth_frame, origin xyz=0 0 0 rpy=0 0 0
- added joint d455_depth_optical_joint: type fixed, parent d455_depth_frame, child d455_depth_optical_frame, origin xyz=0 0 0 rpy=-1.5707963 0 -1.5707963
- added joint d455_infra1_joint: type fixed, parent d455_link, child d455_infra1_frame, origin xyz=0 0 0 rpy=0 0 0
- added joint d455_infra1_optical_joint: type fixed, parent d455_infra1_frame, child d455_infra1_optical_frame, origin xyz=0 0 0 rpy=-1.5707963 0 -1.5707963
- added joint d455_infra2_joint: type fixed, parent d455_link, child d455_infra2_frame, origin xyz=0 -0.095 0 rpy=0 0 0
- added joint d455_infra2_optical_joint: type fixed, parent d455_infra2_frame, child d455_infra2_optical_frame, origin xyz=0 0 0 rpy=-1.5707963 0 -1.5707963
- added joint d455_joint: type fixed, parent base_link, child d455_link, origin xyz=0.29 0.0475 1.69 rpy=0 0.1745329 0

Commit message: alfred: use the solved d455 mount instead of the photo estimate
Registering the D455 depth against the point-lio lidar map on
drive_2026-08-18_23-05-04 moves the camera 15 cm down and 7 cm back from the
value scaled off the side photo, and cuts median error from 5.6 to 3.1 cm.

File: dimos/robot/diy/alfred/alfred.urdf (robot description, URDF)
Before this commit: robot alfred, 30 links, 29 joints
Joints:
- joint d455_joint: origin xyz=0.29 0.0475 1.69 rpy=0 0.1745329 0 -> xyz=0.2146 -0.0008 1.5435 rpy=0.0012 0.1448 -0.0106

Commit message: alfred: add alfred-mls-nav-lidar for multi-IMU dimSLAM
The raw Livox driver replaces Point-LIO so the Mid-360's own IMU reaches
dimSLAM's fusion alongside the D455's, and the voxel map raytraces the
lidar cloud instead of D455 depth. Only one process can hold the lidar's
host endpoint, and the raw driver is the one that publishes the IMU;
Point-LIO's lidar odometry is what dimSLAM is replacing anyway.

File: dimos/robot/diy/alfred/alfred.urdf (robot description, URDF)
Before this commit: robot alfred, 30 links, 29 joints
Links:
- added link mid360_imu_link
Joints:
- added joint mid360_imu_joint: type fixed, parent mid360_link, child mid360_imu_link, origin xyz=0.011 0.02329 -0.04412 rpy=0 0 0
